Commit message: Add panda gripper planning and execution support

File: src/abb_irb140_moveit_config/config/abb_irb140.ros2_control.xacro (robot description, xacro)
@@ -50,4 +50,11 @@
                 <state_interface name="velocity"/>
             </joint>
+            <joint name="gripper_finger_joint1">
+                <command_interface name="position"/>
+                <state_interface name="position">
+                  <param name="initial_value">${initial_positions['gripper_finger_joint1']}</param>
+                </state_interface>
+                <state_interface name="velocity"/>
+            </joint>
         </ros2_control>
     </xacro:macro>

File: src/abb_irb140_moveit_config/config/abb_irb140.urdf.xacro (robot description, xacro)
@@ -4,3 +4,6 @@
     <!-- Import abb_irb140 urdf file -->
     <xacro:include filename="$(find abb_irb140_support)/urdf/irb140.xacro" />
+    <!-- Import control_xacro -->
+    <xacro:include filename="abb_irb140.ros2_control.xacro" />
+    <xacro:abb_irb140_ros2_control name="FakeSystem" initial_positions_file="$(arg initial_positions_file)"/>
 </robot>
