Commit message: Working prototype side-grasp pick and place demo

File: src/abb_irb140_moveit_config/config/abb_irb140.urdf.xacro (robot description, xacro)
@@ -4,6 +4,13 @@
     <!-- Import abb_irb140 urdf file -->
     <xacro:include filename="$(find abb_irb140_support)/urdf/irb140.xacro" />
+<!--
+  Disabled for this project.
+  abb_irb140_support/urdf/irb140.xacro already provides the real/control-ready
+  ros2_control block named IRB140System.
+  Leaving the MoveIt-generated FakeSystem enabled creates duplicate command
+  interfaces such as gripper_finger_joint1/position.
+-->
     <!-- Import control_xacro -->
-    <xacro:include filename="abb_irb140.ros2_control.xacro" />
-    <xacro:abb_irb140_ros2_control name="FakeSystem" initial_positions_file="$(arg initial_positions_file)"/>
+    <!--<xacro:include filename="abb_irb140.ros2_control.xacro" />-->
+    <!--<xacro:abb_irb140_ros2_control name="FakeSystem" initial_positions_file="$(arg initial_positions_file)"/>-->
 </robot>

File: src/abb_irb140_support/urdf/grippers/panda_gripper_macro.xacro (robot description, xacro)
@@ -55,4 +55,11 @@
       <limit lower="0.0" upper="0.04" effort="100" velocity="0.2"/>
     </joint>
+    <!-- Grasp frame: center point between the fingers where objects are attached -->
+    <link name="${prefix}grasp_frame"/>
+    <joint name="${prefix}grasp_frame_joint" type="fixed">
+      <parent link="${prefix}panda_hand"/>
+      <child link="${prefix}grasp_frame"/>
+      <origin xyz="0 0 0.085" rpy="0 0 0"/>
+    </joint>
     <!-- Right finger joint -->
     <joint name="${prefix}finger_joint2" type="prismatic">
