Commit message: Stabilize Gazebo control for IRB140

File: src/abb_irb140_support/urdf/grippers/panda_gripper_macro.xacro (robot description, xacro)
@@ -20,4 +20,5 @@
         </geometry>
       </collision>
+    <xacro:box_inertial mass="1.0" x="0.10" y="0.08" z="0.08"/>
     </link>
     <!-- Left finger -->
@@ -33,4 +34,5 @@
         </geometry>
       </collision>
+    <xacro:box_inertial mass="0.10" x="0.02" y="0.02" z="0.08"/>
     </link>
     <!-- Right finger -->
@@ -46,4 +48,5 @@
         </geometry>
       </collision>
+    <xacro:box_inertial mass="0.10" x="0.02" y="0.02" z="0.08"/>
     </link>
     <!-- Left finger joint -->

File: src/abb_irb140_support/urdf/irb140.xacro (robot description, xacro)
@@ -1,9 +1,16 @@
 <?xml version="1.0" ?>
 <robot name="abb_irb140" xmlns:xacro="http://ros.org/wiki/xacro">
+        <xacro:arg name="use_gazebo" default="false"/>
 	<xacro:include filename="$(find abb_irb140_support)/urdf/irb140_macro.xacro"/>
 	<xacro:abb_irb140 prefix=""/>
 <ros2_control name="IRB140System" type="system">
   <hardware>
-    <plugin>mock_components/GenericSystem</plugin>
+    <xacro:if value="$(arg use_gazebo)">
+      <plugin>gz_ros2_control/GazeboSimSystem</plugin>
+      <param name="position_proportional_gain">0.8</param>
+    </xacro:if>
+    <xacro:unless value="$(arg use_gazebo)">
+      <plugin>mock_components/GenericSystem</plugin>
+    </xacro:unless>
   </hardware>
   <joint name="joint_1">
@@ -43,3 +50,23 @@
   </joint>
 </ros2_control>
+<xacro:if value="$(arg use_gazebo)">
+  <!--
+    Gazebo-only temporary mounting fix.
+    This represents the industrial robot being bolted to the world/floor.
+    Long-term, this should move into a proper Gazebo workcell/world model.
+  -->
+  <gazebo>
+    <joint name="world_to_base_link" type="fixed">
+      <parent>world</parent>
+      <child>base_link</child>
+    </joint>
+  </gazebo>
+  <gazebo>
+    <plugin
+      filename="libgz_ros2_control-system.so"
+      name="gz_ros2_control::GazeboSimROS2ControlPlugin">
+      <parameters>$(find abb_irb140_moveit_config)/config/ros2_controllers.yaml</parameters>
+    </plugin>
+  </gazebo>
+</xacro:if>
 </robot>

File: src/abb_irb140_support/urdf/irb140_macro.xacro (robot description, xacro)
@@ -2,4 +2,23 @@
 <robot xmlns:xacro="http://ros.org/wiki/xacro">
 <xacro:include filename="$(find abb_irb140_support)/urdf/grippers/panda_gripper_macro.xacro"/>
+<!--
+  Approximate inertial model for Gazebo simulation.
+  These values are not manufacturer-accurate ABB dynamics.
+  They are conservative box approximations so Gazebo can create
+  physically valid links.
+-->
+<xacro:macro name="box_inertial" params="mass x y z">
+  <inertial>
+    <origin xyz="0 0 0" rpy="0 0 0"/>
+    <mass value="${mass}"/>
+    <inertia
+      ixx="${mass * (y * y + z * z) / 12.0}"
+      ixy="0.0"
+      ixz="0.0"
+      iyy="${mass * (x * x + z * z) / 12.0}"
+      iyz="0.0"
+      izz="${mass * (x * x + y * y) / 12.0}"/>
+  </inertial>
+</xacro:macro>
 <xacro:macro name="abb_irb140" params="prefix">
     <!-- link list -->
@@ -22,4 +41,5 @@
       </material>
     </collision>
+    <xacro:box_inertial mass="20.0" x="0.35" y="0.35" z="0.30"/>
   </link>
   <link name="${prefix}link_1">
@@ -38,4 +58,5 @@
       <material name="yellow"/>
     </collision>
+    <xacro:box_inertial mass="12.0" x="0.30" y="0.30" z="0.35"/>
   </link>
   <link name="${prefix}link_2">
@@ -54,4 +75,5 @@
       <material name="yellow"/>
     </collision>
+    <xacro:box_inertial mass="18.0" x="0.18" y="0.20" z="0.50"/>
   </link>
   <link name="${prefix}link_3">
@@ -70,4 +92,5 @@
       <material name="yellow"/>
     </collision>
+    <xacro:box_inertial mass="10.0" x="0.22" y="0.18" z="0.35"/>
   </link>
   <link name="${prefix}link_4">
@@ -86,4 +109,5 @@
       <material name="yellow"/>
     </collision>
+    <xacro:box_inertial mass="6.0" x="0.25" y="0.14" z="0.14"/>
   </link>
   <link name="${prefix}link_5">
@@ -102,4 +126,5 @@
       <material name="yellow"/>
     </collision>
+    <xacro:box_inertial mass="4.0" x="0.16" y="0.12" z="0.12"/>
   </link>
   <link name="${prefix}link_6">
@@ -118,4 +143,5 @@
       <material name="yellow"/>
     </collision>
+    <xacro:box_inertial mass="2.0" x="0.12" y="0.10" z="0.10"/>
   </link>
   <link name="${prefix}tool0"/>
@@ -127,5 +153,5 @@
     <child link="${prefix}link_1"/>
     <axis xyz="0 0 1"/>
-    <limit effort="0" lower="-3.1416" upper="3.1416" velocity="2.618"/>
+    <limit effort="200" lower="-3.1416" upper="3.1416" velocity="2.618"/>
   </joint>
   <joint name="joint_2" type="revolute">
@@ -134,5 +160,5 @@
     <child link="${prefix}link_2"/>
     <axis xyz="0 1 0"/>
-    <limit effort="0" lower="-1.7453" upper="1.7453" velocity="2.618"/>
+    <limit effort="250" lower="-1.7453" upper="1.7453" velocity="2.618"/>
   </joint>
   <joint name="joint_3" type="revolute">
@@ -141,5 +167,5 @@
     <child link="${prefix}link_3"/>
     <axis xyz="0 1 0"/>
-    <limit effort="0" lower="-2.4434" upper="2.4434" velocity="2.618"/>
+    <limit effort="200" lower="-2.4434" upper="2.4434" velocity="2.618"/>
   </joint>
   <joint name="${prefix}joint_4" type="revolute">
@@ -148,5 +174,5 @@
     <child link="${prefix}link_4"/>
     <axis xyz="1 0 0"/>
-    <limit effort="0" lower="-3.49" upper="3.49" velocity="6.2832"/>
+    <limit effort="80" lower="-3.49" upper="3.49" velocity="6.2832"/>
   </joint>
   <joint name="${prefix}joint_5" type="revolute">
@@ -155,5 +181,5 @@
     <child link="${prefix}link_5"/>
     <axis xyz="0 1 0"/>
-    <limit effort="0" lower="-2.0071" upper="2.0071" velocity="6.2832"/>
+    <limit effort="60" lower="-2.0071" upper="2.0071" velocity="6.2832"/>
   </joint>
   <joint name="${prefix}joint_6" type="revolute">
@@ -162,5 +188,5 @@
     <child link="${prefix}link_6"/>
     <axis xyz="1 0 0"/>
-    <limit effort="0" lower="-6.9813" upper="6.9813" velocity="7.854"/>
+    <limit effort="40" lower="-6.9813" upper="6.9813" velocity="7.854"/>
   </joint>
   <joint name="${prefix}joint_6-tool0" type="fixed">
