Commit message: Added panda gripper and fixed ros2_control issues

File: src/abb_irb140_support/urdf/irb140.xacro (robot description, xacro)
@@ -37,4 +37,9 @@
     <state_interface name="velocity"/>
   </joint>
+  <joint name="gripper_finger_joint1">
+    <command_interface name="position"/>
+    <state_interface name="position"/>
+    <state_interface name="velocity"/>
+  </joint>
 </ros2_control>
 </robot>

File: src/abb_irb140_support/urdf/irb140_macro.xacro (robot description, xacro)
@@ -1,4 +1,5 @@
 <?xml version="1.0"?>
 <robot xmlns:xacro="http://ros.org/wiki/xacro">
+<xacro:include filename="$(find abb_irb140_support)/urdf/grippers/panda_gripper_macro.xacro"/>
 <xacro:macro name="abb_irb140" params="prefix">
     <!-- link list -->
@@ -168,4 +169,7 @@
     <origin rpy="0 0 0" xyz="0 0 0"/>
   </joint>
+  <xacro:panda_gripper
+    parent="${prefix}tool0"
+    prefix="gripper_"/>
     <!-- end of joint list -->
     <!-- ROS base_link to ABB World Coordinates transform -->

Commit message: Restore stable Gazebo simulation baseline

File: src/abb_irb140_support/urdf/irb140.xacro (robot description, xacro)
@@ -49,17 +49,27 @@
     <state_interface name="velocity"/>
   </joint>
+  <!--
+    State-only mimic finger for Gazebo.
+    gripper_finger_joint1 is the commanded joint.
+    gripper_finger_joint2 already has a URDF <mimic> tag in the gripper macro.
+    For gz_ros2_control, the mimic joint must not have a command interface.
+  -->
+  <joint name="gripper_finger_joint2">
+    <state_interface name="position"/>
+    <state_interface name="velocity"/>
+  </joint>
 </ros2_control>
 <xacro:if value="$(arg use_gazebo)">
   <!--
-    Gazebo-only temporary mounting fix.
-    This represents the industrial robot being bolted to the world/floor.
-    Long-term, this should move into a proper Gazebo workcell/world model.
+    Massless world root used in Gazebo mode.
+    This prevents KDL from treating base_link, which has inertia, as the
+    root link of the robot tree.
   -->
-  <gazebo>
-    <joint name="world_to_base_link" type="fixed">
-      <parent>world</parent>
-      <child>base_link</child>
-    </joint>
-  </gazebo>
+  <link name="world"/>
+  <joint name="world_to_base_link" type="fixed">
+    <parent link="world"/>
+    <child link="base_link"/>
+    <origin xyz="0 0 0" rpy="0 0 0"/>
+  </joint>
   <gazebo>
     <plugin
